File: kicad/Anemometr_v3/Anemometr.sch (KiCad schematic (older format))
At the start: 150 parts, among them J1 TxD, J10 +Z1, J11 +Z2, J12 +Z3, J13 +Z4, J14 -Z1, J15 -Z2, J16 -Z3, J17 -Z4, J18 1 TxD+, J19 2 TxD-, J2 RxD, J20 3 RxD+, J21 4-5, J22 6 RxD-, J23 7-8, J24 Conn_01x01_Female, J25 Conn_01x01_Female, J3 SCL, J4 SDA, J5 RST, J6 +EXT, J7 -EXT, J8 SWD, J9 SWC, Q1 5N10, U1 STM32F103C8Tx, U2 TS5A3166DBVR, U3 TS5A3166DBVR, U4 LMR14206, U6 NCP1117-3.3, U8 TLV3201DBV, U9 MCP1703-3.3, Y1 CSTCE8M00G52A-R0, Y2 ECS-250-20-33

Commit message: изменено:      kicad/Anemometr_v3/Anemometr-cache.lib 	изменено:      kicad/Anemometr_v3/Anemometr.kicad_pcb 	изменено:      kicad/Anemometr_v3/Anemometr.kicad_pcb-bak 	изменено:      kicad/Anemometr_v3/Anemometr.sch 	изменено:      kicad/Anemometr_v3/Anemometr.sch-bak 	новый файл:    stm32cubeide/Anemometer/Debug/Core/Src/dhcp.d 	новый файл:    stm32cubeide/Anemometer/Debug/Core/Src/dhcp.o 	новый файл:    stm32cubeide/Anemometer/Debug/Core/Src/dhcp.su 	новый файл:    stm32cubeide/Anemometer/Debug/Core/Src/dns.d 	новый файл:    stm32cubeide/Anemometer/Debug/Core/Src/dns.o 	новый файл:    stm32cubeide/Anemometer/Debug/Core/Src/dns.su 	новый файл:    stm32cubeide/Anemometer/Debug/Core/Src/socket.d 	новый файл:    stm32cubeide/Anemometer/Debug/Core/Src/socket.o 	новый файл:    stm32cubeide/Anemometer/Debug/Core/Src/socket.su 	новый файл:    stm32cubeide/Anemometer/Debug/Core/Src/w5500.d 	новый файл:    stm32cubeide/Anemometer/Debug/Core/Src/w5500.o 	новый файл:    stm32cubeide/Anemometer/Debug/Core/Src/w5500.su 	новый файл:    stm32cubeide/Anemometer/Debug/Core/Src/wizchip_conf.d 	новый файл:    stm32cubeide/Anemometer/Debug/Core/Src/wizchip_conf.o 	новый файл:    stm32cubeide/Anemometer/Debug/Core/Src/wizchip_conf.su 	новый файл:    stm32cubeide/Anemometer/Debug/Drivers/STM32F1xx_HAL_Driver/Src/stm32f1xx_hal_i2c.d 	новый файл:    stm32cubeide/Anemometer/Debug/Drivers/STM32F1xx_HAL_Driver/Src/stm32f1xx_hal_i2c.o 	новый файл:    stm32cubeide/Anemometer/Debug/Drivers/STM32F1xx_HAL_Driver/Src/stm32f1xx_hal_i2c.su 	новый файл:    stm32cubeide/Anemometer/Drivers/STM32F1xx_HAL_Driver/Inc/stm32f1xx_hal_iwdg.h 	новый файл:    stm32cubeide/Anemometer/Drivers/STM32F1xx_HAL_Driver/Inc/stm32f1xx_hal_spi.h 	новый файл:    stm32cubeide/Anemometer/Drivers/STM32F1xx_HAL_Driver/Src/stm32f1xx_hal_iwdg.c 	новый файл:    stm32cubeide/Anemometer/Drivers/STM32F1xx_HAL_Driver/Src/stm32f1xx_hal_spi.c 	новый файл:    stm32cubeide/Anemometer/Release/Anemometer.hex 	новый файл:    stm32cubeide/A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
Parts:
- removed C40, C41: 390p, Capacitor_SMD:C_0402_1005Metric, symbol Device:C
- removed J8: SWD, My-library:SMD-CONN, symbol Connector:Conn_01x01_Female
- removed J9: SWC, My-library:SMD-CONN, symbol Connector:Conn_01x01_Female
- removed R31: 1.3k, Resistor_SMD:R_0402_1005Metric, symbol Device:R
- added J8: SWD, My-library:SMD-CONN, symbol My_Library:Conn
- added J9: SWC, My-library:SMD-CONN, symbol My_Library:Conn
- C51: footprint Capacitor_SMD:C_0603_1608Metric -> Capacitor_SMD:C_0402_1005Metric
- C53: footprint Capacitor_SMD:C_0603_1608Metric -> Capacitor_SMD:C_0805_2012Metric
- D13, D8: value MBR0540 -> F7
- D16: value MBR0540 -> SS34
- D17: value MBR0540 -> SS56; footprint Diode_SMD:D_SOD-123 -> Diode_SMD:D_SMA
- L5: value CoilCraft HLPS4018-472MR -> 15uH; footprint Inductor_SMD:L_Coilcraft_LPS4018 -> Inductor_SMD:L_Abracon_ASPI-0630LR
- R17: value 110k -> 100k
Connections:
- net labels added: +Z1, +Z2, +Z3, +Z4, Rst, RxD, SCL, SDA, SWC, SWD, TxD
- wire segments 275 -> 288
- no-connect marks 32 -> 31
Other:
- moved on the sheet: C17, C18, C21, C29, C34, C47, C51, C59, D5, D7A, D7B, R13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

Commit message: изменено:      kicad/Anemometr_v2/fp-info-cache 	изменено:      kicad/Anemometr_v3/Anemometr-cache.lib 	изменено:      kicad/Anemometr_v3/Anemometr-rescue.lib 	изменено:      kicad/Anemometr_v3/Anemometr.sch 	изменено:      kicad/Anemometr_v3/Anemometr.sch-bak 	изменено:      stm32cubeide/Anemometer/.settings/language.settings.xml 	Documents/1690.png 	Documents/BST-BME280-DS002-1509607.pdf
Parts:
- D18: symbol My_Library:MC33375ST -> Anemometr-rescue:MC33375ST-My_Library
- J8, J9: symbol My_Library:Conn -> Anemometr-rescue:Conn-My_Library
- R21: value 30k -> 43k
- R25: value 300k -> 100k
Changed lines of the file:
@@
 P 9250 1950
 F 0 "R25" H 9400 1850 50  0000 C CNN
-F 1 "300k" H 9400 1950 50  0000 C CNN
+F 1 "100k" H 9400 1950 50  0000 C CNN
 F 2 "Resistor_SMD:R_0402_1005Metric" V 9180 1950 50  0001 C CNN
 F 3 "~" H 9250 1950 50  0001 C CNN
@@
 P 8750 5650
 F 0 "R21" H 8950 5700 50  0000 R CNN
-F 1 "30k" H 8950 5600 50  0000 R CNN
+F 1 "43k" H 8950 5600 50  0000 R CNN
 F 2 "Resistor_SMD:R_0603_1608Metric" V 8680 5650 50  0001 C CNN
 F 3 "~" H 8750 5650 50  0001 C CNN
@@
 	7850 3450 7850 4900
 $Comp
-L My_Library:MC33375ST D18
+L Anemometr-rescue:MC33375ST-My_Library D18
 U 1 1 634E9456
 P 11000 4400
@@
 $EndComp
 $Comp
-L My_Library:Conn J9
+L Anemometr-rescue:Conn-My_Library J9
 U 1 1 63B27BC5
 P 6000 5650
@@
 $EndComp
 $Comp
-L My_Library:Conn J8
+L Anemometr-rescue:Conn-My_Library J8
 U 1 1 63B4B18F
 P 6000 5550

Commit message: изменено:      kicad/Anemometr_v3/Anemometr-cache.lib 	изменено:      kicad/Anemometr_v3/Anemometr.kicad_pcb 	изменено:      kicad/Anemometr_v3/Anemometr.kicad_pcb-bak 	изменено:      kicad/Anemometr_v3/Anemometr.pro 	изменено:      kicad/Anemometr_v3/Anemometr.sch 	изменено:      kicad/Anemometr_v3/Anemometr.sch-bak 	изменено:      kicad/Anemometr_v3/fp-info-cache
Parts:
- removed R38: 100k, Resistor_SMD:R_0603_1608Metric, symbol Device:R
- removed R39: 3k, Resistor_SMD:R_0603_1608Metric, symbol Device:R
- removed U8: TLV3201DBV, Package_TO_SOT_SMD:SOT-23-5, symbol Comparator:MCP6566
- added C32, C5, C52, C57: 0.1uF, Capacitor_SMD:C_0402_1005Metric, symbol Device:C
- added C40: 100nF, Capacitor_SMD:C_0402_1005Metric, symbol Device:C
- added C41: 1,5nF, Capacitor_SMD:C_0402_1005Metric, symbol Device:C
- added C6: 10nF, Capacitor_SMD:C_0402_1005Metric, symbol Device:C
- added C60, C61: 10uF, Capacitor_SMD:C_0805_2012Metric, symbol Device:C
- added D19: MAX4477, Package_SO:MSOP-8_3x3mm_P0.65mm, symbol Anemometr-rescue:MAX4477-My_Library
- added D20, D21: TLV3501, Package_TO_SOT_SMD:SOT-23-6, symbol My_Library:TLV3501-2
- added J26: Conn_01x01_Female, My-library:ConnMini, symbol Connector:Conn_01x01_Female
- added R31: 20k, Resistor_SMD:R_0402_1005Metric, symbol Device:R
- added R45: 1k, Resistor_SMD:R_0402_1005Metric, symbol Device:R
- added R46, R48, R50: 100k, Resistor_SMD:R_0402_1005Metric, symbol Device:R
- added R47: 5.1k, Resistor_SMD:R_0402_1005Metric, symbol Device:R
- added R49: 10k, Resistor_SMD:R_0402_1005Metric, symbol Device:R
- added R51: 3k, Resistor_SMD:R_0402_1005Metric, symbol Device:R
- added R7, R8: 3k, Resistor_SMD:R_0603_1608Metric, symbol Device:R
- added U5, U7: TS5A3166DBVR, Package_TO_SOT_SMD:SOT-23-5, symbol Analog_Switch:TS5A3166DBVR
- added U8: MCP1703-3.3, Package_TO_SOT_SMD:SOT-23, symbol Regulator_Linear:MCP1700-3302E_SOT23
- C1, C2: footprint Capacitor_SMD:C_0805_2012Metric -> Capacitor_SMD:C_0402_1005Metric
- C42, C45, C46, C47, C48, C59: footprint Capacitor_SMD:C_0603_1608Metric -> Capacitor_SMD:C_0402_1005Metric
- C55: footprint Capacitor_SMD:C_0805_2012Metric -> Capacitor_SMD:C_0603_1608Metric
- J1, J2, J24, J25, J3, J4, J5, J8, J9: footprint My-library:SMD-CONN -> My-library:ConnMini
- R17: value 100k -> 110k
- R32, R35, R36, R37, R40, R5: footprint Resistor_SMD:R_0603_1608Metric -> Resistor_SMD:R_0402_1005Metric
Connections:
- net labels added: +3.3VP, SInput, Z1-2, Z3, Z3-4, Z4, a, swc, swd
- net labels removed: Analog, SWC, SWD, SensorInput
- wire segments 288 -> 323
- no-connect marks 31 -> 23
Other:
- moved on the sheet: C1, C10, C11, C12, C13, C14, C15, C16, C17, C18, C19, C2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

Commit message: изменено:      kicad/Anemometr_v3/Anemometr.kicad_pcb 	изменено:      kicad/Anemometr_v3/Anemometr.kicad_pcb-bak 	изменено:      kicad/Anemometr_v3/Anemometr.sch 	изменено:      kicad/Anemometr_v3/Anemometr.sch-bak
Connections:
- net 12-16v renamed 12v
- net 5.6-6v renamed 6v
Other:
- moved on the sheet: C22, C23, C30, C36, C37, C53, C54, C55, C56, C58, C60, C61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

Commit message: изменено:      kicad/Anemometr_v3/Anemometr.pdf 	изменено:      kicad/Anemometr_v3/Anemometr.sch 	изменено:      kicad/Anemometr_v3/Anemometr.sch-bak
Parts:
- D11: value SD4932B -> U6119SA
Changed lines of the file:
@@
 P 8150 6950
 F 0 "D11" H 8150 7365 50  0000 C CNN
-F 1 "SD4932B" H 8150 7274 50  0000 C CNN
+F 1 "U6119SA" H 8150 7274 50  0000 C CNN
 F 2 "Package_SO:SOIC-8-N7_3.9x4.9mm_P1.27mm" H 8100 6850 50  0001 C CNN
 F 3 "" H 8100 6850 50  0001 C CNN

Commit message: изменено:      kicad/Anemometr_v3/Anemometr-cache.lib 	изменено:      kicad/Anemometr_v3/Anemometr-rescue.lib 	изменено:      kicad/Anemometr_v3/Anemometr.sch 	изменено:      kicad/Anemometr_v3/Anemometr.sch-bak 	изменено:      stm32cubeide/Anemometer/.settings/language.settings.xml
Parts:
- D20, D21: symbol My_Library:TLV3501-2 -> Anemometr-rescue:TLV3501-2-My_Library
Changed lines of the file:
@@
 Connection ~ 5900 3950
 $Comp
-L My_Library:TLV3501-2 D20
+L Anemometr-rescue:TLV3501-2-My_Library D20
 U 1 1 637C998F
 P 10050 1350
@@
 	10150 1600 10200 1600
 $Comp
-L My_Library:TLV3501-2 D21
+L Anemometr-rescue:TLV3501-2-My_Library D21
 U 1 1 638DF360
 P 10050 3150

Commit message: изменено:      kicad/Anemometr_v3/Anemometr-cache.lib 	изменено:      kicad/Anemometr_v3/Anemometr.kicad_pcb 	изменено:      kicad/Anemometr_v3/Anemometr.kicad_pcb-bak 	изменено:      kicad/Anemometr_v3/Anemometr.sch 	изменено:      kicad/Anemometr_v3/Anemometr.sch-bak
Parts:
- removed C1, C17, C2, C21, C32, C5, C51, C52, C57, C59: 0.1uF, Capacitor_SMD:C_0402_1005Metric, symbol Device:C
- removed C18, C6: 10nF, Capacitor_SMD:C_0402_1005Metric, symbol Device:C
- removed C34, C40: 100nF, Capacitor_SMD:C_0402_1005Metric, symbol Device:C
- removed C41, C47: 1,5nF, Capacitor_SMD:C_0402_1005Metric, symbol Device:C
- removed C60, C61: 10uF, Capacitor_SMD:C_0805_2012Metric, symbol Device:C
- removed D19, D7: MAX4477, Package_SO:MSOP-8_3x3mm_P0.65mm, symbol Anemometr-rescue:MAX4477-My_Library
- removed D20, D21: TLV3501, Package_TO_SOT_SMD:SOT-23-6, symbol Anemometr-rescue:TLV3501-2-My_Library
- removed R13, R31: 20k, Resistor_SMD:R_0402_1005Metric, symbol Device:R
- removed R16, R25, R33, R46, R48, R50: 100k, Resistor_SMD:R_0402_1005Metric, symbol Device:R
- removed R17: 110k, Resistor_SMD:R_0402_1005Metric, symbol Device:R
- removed R20, R45: 1k, Resistor_SMD:R_0402_1005Metric, symbol Device:R
- removed R29, R47: 5.1k, Resistor_SMD:R_0402_1005Metric, symbol Device:R
- removed R37, R49: 10k, Resistor_SMD:R_0402_1005Metric, symbol Device:R
- removed R5, R51: 3k, Resistor_SMD:R_0402_1005Metric, symbol Device:R
- removed R6, R7, R8: 3k, Resistor_SMD:R_0603_1608Metric, symbol Device:R
- removed U2, U3, U5, U7: TS5A3166DBVR, Package_TO_SOT_SMD:SOT-23-5, symbol Analog_Switch:TS5A3166DBVR
- removed U8: MCP1703-3.3, Package_TO_SOT_SMD:SOT-23, symbol Regulator_Linear:MCP1700-3302E_SOT23
- added J27, J28, J29, J30, J31, J32, J33, J34, J35, J36, J37, J38, J39: +Z1, My-library:SMD-CONN, symbol Connector:Conn_01x01_Female
- J24, J25, J26: value Conn_01x01_Female -> +Z1; footprint My-library:ConnMini -> My-library:SMD-CONN
Connections:
- net +5VA: now also J24.1 (Pin_1), J25.1 (Pin_1), J26.1 (Pin_1), J27.1 (Pin_1)
- net GND: now also J36.1 (Pin_1), J37.1 (Pin_1), J38.1 (Pin_1), J39.1 (Pin_1)
- net SInput renamed SIn
- net SIn: now also J28.1 (Pin_1), J29.1 (Pin_1), J30.1 (Pin_1), J31.1 (Pin_1); no longer J24.1 (Pin_1)
- net Z1 renamed Z1Sel
- net Z1Sel: now also J32.1 (Pin_1)
- net Z1-2: no longer names the net of U1.3 (PC14)
- net Z2 renamed Z2Sel
- net Z2Sel: now also J33.1 (Pin_1)
- net Z3 renamed Z3Sel
- net Z3Sel: now also J34.1 (Pin_1)
- net Z3-4: no longer names the net of U1.2 (PC13)
- net Z4 renamed Z4Sel
- net Z4Sel: now also J35.1 (Pin_1)
- no-connect marks 23 -> 28
Other:
- moved on the sheet: C11, C13, C22, C23, C3, C30, C36, C37, C53, C54, C55, C56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

Commit message: изменено:      kicad/Anemometr_v3/Anemometr.sch 	изменено:      kicad/Anemometr_v3/Anemometr.sch-bak
Parts:
- D17: value SS56 -> SS56, VS10MQ060-M3/5
Changed lines of the file:
@@
 P 9300 5150
 F 0 "D17" V 9300 5300 50  0000 C CNN
-F 1 "SS56" V 9650 5150 50  0001 C CNN
+F 1 "SS56, VS10MQ060-M3/5" V 9650 5150 50  0001 C CNN
 F 2 "Diode_SMD:D_SMA" H 9300 5150 50  0001 C CNN
 F 3 "~" H 9300 5150 50  0001 C CNN
