File: kicad/Amp/Amp.sch (KiCad schematic (older format))
At the start: 23 parts, among them J1 Conn, J2 Conn, J3 Conn, J4 Conn, J5 Conn, J6 Conn, Q1 Q_NPN_BEC, U1 AD8541, U2 TS5A3166DBVR, U3 MCP1700

Commit message: изменено:      kicad/Amp/Amp-cache.lib 	изменено:      kicad/Amp/Amp.kicad_pcb 	изменено:      kicad/Amp/Amp.kicad_pcb-bak 	изменено:      kicad/Amp/Amp.sch 	изменено:      kicad/Amp/Amp.sch-bak 	изменено:      stm32cubeide/Anemometr_v3/Core/Src/main.c 	изменено:      stm32cubeide/Anemometr_v3/Core/Src/stm32f1xx_it.c 	изменено:      stm32cubeide/Anemometr_v3/Debug/Anemometr_3.bin 	изменено:      stm32cubeide/Anemometr_v3/Debug/Anemometr_3.elf 	изменено:      stm32cubeide/Anemometr_v3/Debug/Anemometr_3.list 	изменено:      stm32cubeide/Anemometr_v3/Debug/Anemometr_3.map 	изменено:      stm32cubeide/Anemometr_v3/Debug/Core/Src/main.o 	изменено:      stm32cubeide/Anemometr_v3/Debug/Core/Src/main.su 	изменено:      stm32cubeide/Anemometr_v3/Debug/Core/Src/stm32f1xx_it.o 	изменено:      stm32cubeide/Anemometr_v3/Release/Anemometr_3.bin 	изменено:      stm32cubeide/Anemometr_v3/Release/Anemometr_3.elf 	изменено:      stm32cubeide/Anemometr_v3/Release/Anemometr_3.list 	изменено:      stm32cubeide/Anemometr_v3/Release/Anemometr_3.map 	изменено:      stm32cubeide/Anemometr_v3/Release/Core/Src/main.o 	изменено:      stm32cubeide/Anemometr_v3/Release/Core/Src/main.su 	изменено:      stm32cubeide/Anemometr_v3/Release/Core/Src/stm32f1xx_it.o
Parts:
- added J7: Conn, My-library:SMD-CONN, symbol Amp-rescue:Conn-My_Library
- added U4: TS5A3167DBVR, Package_TO_SOT_SMD:SOT-23-5, symbol My_Library:TS5A3167DBVR
- C1: footprint Capacitor_SMD:C_0603_1608Metric -> Resistor_SMD:R_0603_1608Metric
- J1, J2: footprint Connector_Pin:Pin_D0.7mm_L6.5mm_W1.8mm_FlatFork -> My-library:connBig; symbol My_Library:Conn -> Amp-rescue:Conn-My_Library
- J3, J4, J5, J6: symbol My_Library:Conn -> Amp-rescue:Conn-My_Library
Connections:
- net labels added: 3.3v, Signal
- wire segments 35 -> 51
Other:
- moved on the sheet: C3, R6, U2
Changed lines of the file:
@@
 $EndDescr
 $Comp
-L My_Library:Conn J1
+L Amp-rescue:Conn-My_Library J1
 U 1 1 63C7E189
-P 4450 2750
-F 0 "J1" H 4392 2565 50  0001 C CNN
-F 1 "Conn" H 4392 2656 50  0001 C CNN
-F 2 "Connector_Pin:Pin_D0.7mm_L6.5mm_W1.8mm_FlatFork" H 4500 2600 50  0001 C CNN
-F 3 "~" H 4450 2750 50  0001 C CNN
-	1    4450 2750
+P 3400 2350
+F 0 "J1" H 3342 2165 50  0001 C CNN
+F 1 "Conn" H 3342 2256 50  0001 C CNN
+F 2 "My-library:connBig" H 3450 2200 50  0001 C CNN
+F 3 "~" H 3400 2350 50  0001 C CNN
+	1    3400 2350
 	-1   0    0    1
 $EndComp
@@
 $EndComp
 $Comp
-L My_Library:Conn J2
+L Amp-rescue:Conn-My_Library J2
 U 1 1 63C7FD46
-P 4450 3150
-F 0 "J2" H 4392 2965 50  0001 C CNN
-F 1 "Conn" H 4392 3056 50  0001 C CNN
-F 2 "Connector_Pin:Pin_D0.7mm_L6.5mm_W1.8mm_FlatFork" H 4500 3000 50  0001 C CNN
-F 3 "~" H 4450 3150 50  0001 C CNN
-	1    4450 3150
+P 3400 3150
+F 0 "J2" H 3342 2965 50  0001 C CNN
+F 1 "Conn" H 3342 3056 50  0001 C CNN
+F 2 "My-library:connBig" H 3450 3000 50  0001 C CNN
+F 3 "~" H 3400 3150 50  0001 C CNN
+	1    3400 3150
 	-1   0    0    1
 $EndComp
 $Comp
-L My_Library:Conn J6
+L Amp-rescue:Conn-My_Library J6
 U 1 1 63C80349
-P 7100 3150
-F 0 "J6" H 7128 3196 50  0001 L CNN
-F 1 "Conn" H 7128 3105 50  0001 L CNN
-F 2 "My-library:SMD-CONN" H 7150 3000 50  0001 C CNN
-F 3 "~" H 7100 3150 50  0001 C CNN
-	1    7100 3150
+P 7400 3150
+F 0 "J6" H 7428 3196 50  0001 L CNN
+F 1 "Conn" H 7428 3105 50  0001 L CNN
+F 2 "My-library:SMD-CONN" H 7450 3000 50  0001 C CNN
+F 3 "~" H 7400 3150 50  0001 C CNN
+	1    7400 3150
 	1    0    0    -1
 $EndComp
@@
 L Device:C C3
 U 1 1 63C8351B
-P 5000 3000
-F 0 "C3" H 4750 3050 50  0000 L CNN
-F 1 "1uF" H 4750 2950 50  0000 L CNN
-F 2 "Capacitor_SMD:C_0603_1608Metric" H 5038 2850 50  0001 C CNN
-F 3 "~" H 5000 3000 50  0001 C CNN
-	1    5000 3000
+P 5100 3000
+F 0 "C3" H 4850 3050 50  0000 L CNN
+F 1 "1uF" H 4850 2950 50  0000 L CNN
+F 2 "Capacitor_SMD:C_0603_1608Metric" H 5138 2850 50  0001 C CNN
+F 3 "~" H 5100 3000 50  0001 C CNN
+	1    5100 3000
 	1    0    0    -1
 $EndComp
@@
 F 0 "C1" V 4450 2750 50  0000 C CNN
 F 1 "1.5n" V 4550 2750 50  0000 C CNN
-F 2 "Capacitor_SMD:C_0603_1608Metric" H 4738 2600 50  0001 C CNN
+F 2 "Resistor_SMD:R_0603_1608Metric" H 4738 2600 50  0001 C CNN
 F 3 "~" H 4700 2750 50  0001 C CNN
 	1    4700 2750
@@
 Wire Wire Line
 	5250 2550 5250 2850
-Wire Wire Line
-	5000 2850 5250 2850
 Connection ~ 5250 2850
-Wire Wire Line
-	5000 3150 5250 3150
 Wire Wire Line
 	5250 3150 5250 3250
@@
 $EndComp
 $Comp
-L My_Library:Conn J3
+L Amp-rescue:Conn-My_Library J3
 U 1 1 63C8F41C
 P 7850 2000
@@
 $EndComp
 $Comp
-L My_Library:Conn J5
+L Amp-rescue:Conn-My_Library J5
 U 1 1 63C8F7BE
-P 7100 2650
-F 0 "J5" H 7128 2696 50  0001 L CNN
-F 1 "Conn" H 7128 2605 50  0001 L CNN
-F 2 "My-library:SMD-CONN" H 7150 2500 50  0001 C CNN
-F 3 "~" H 7100 2650 50  0001 C CNN
-	1    7100 2650
-	1    0    0    -1
-$EndComp
-$Comp
-L My_Library:Conn J4
+P 7400 2650
+F 0 "J5" H 7428 2696 50  0001 L CNN
+F 1 "Conn" H 7428 2605 50  0001 L CNN
+F 2 "My-library:SMD-CONN" H 7450 2500 50  0001 C CNN
+F 3 "~" H 7400 2650 50  0001 C CNN
+	1    7400 2650
+	1    0    0    -1
+$EndComp
+$Comp
+L Amp-rescue:Conn-My_Library J4
 U 1 1 63C92E60
-P 7100 3000
-F 0 "J4" H 7128 3046 50  0001 L CNN
-F 1 "Conn" H 7128 2955 50  0001 L CNN
-F 2 "My-library:SMD-CONN" H 7150 2850 50  0001 C CNN
-F 3 "~" H 7100 3000 50  0001 C CNN
-	1    7100 3000
+P 7400 3000
+F 0 "J4" H 7428 3046 50  0001 L CNN
+F 1 "Conn" H 7428 2955 50  0001 L CNN
+F 2 "My-library:SMD-CONN" H 7450 2850 50  0001 C CNN
+F 3 "~" H 7400 3000 50  0001 C CNN
+	1    7400 3000
 	1    0    0    -1
 $EndComp
@@
 	5150 2750 5400 2750
 Connection ~ 5400 2750
-Wire Wire Line
-	4550 3150 5000 3150
-Connection ~ 5000 3150
 $Comp
 L Device:R R2
@@
 L Analog_Switch:TS5A3166DBVR U2
 U 1 1 63CAD01E
-P 6700 2650
-F 0 "U2" H 6600 2800 50  0000 L CNN
-F 1 "TS5A3166DBVR" H 6900 2550 50  0000 L CNN
-F 2 "Package_TO_SOT_SMD:SOT-23-5" H 6650 2500 50  0001 C CNN
-F 3 " http://www.ti.com/lit/ds/symlink/ts5a3166.pdf" H 6700 2750 50  0001 C CNN
-	1    6700 2650
-	1    0    0    -1
+P 6900 2650
+F 0 "U2" H 6800 2800 50  0000 L CNN
+F 1 "TS5A3166DBVR" H 6650 2050 50  0000 L CNN
+F 2 "Package_TO_SOT_SMD:SOT-23-5" H 6850 2500 50  0001 C CNN
+F 3 " http://www.ti.com/lit/ds/symlink/ts5a3166.pdf" H 6900 2750 50  0001 C CNN
+	1    6900 2650
+	-1   0    0    -1
 $EndComp
 Wire Wire Line
@@
 Wire Wire Line
 	6350 2750 6350 3000
-Wire Wire Line
-	6350 3000 7000 3000
 Connection ~ 6350 2750
 Wire Wire Line
 	6800 2950 6800 3150
 Wire Wire Line
-	6800 3150 7000 3150
+	6800 3150 7300 3150
 Wire Wire Line
 	6550 2000 6650 2000
@@
 Connection ~ 6000 2650
 Wire Wire Line
-	6300 2650 6400 2650
-Wire Wire Line
 	5600 2000 6000 2000
 Connection ~ 5600 2000
@@
 L Device:R R6
 U 1 1 63CF373C
-P 4550 2950
-F 0 "R6" H 4300 3000 50  0000 L CNN
-F 1 "5.1k" H 4300 2900 50  0000 L CNN
-F 2 "Resistor_SMD:R_0603_1608Metric" V 4480 2950 50  0001 C CNN
-F 3 "~" H 4550 2950 50  0001 C CNN
-	1    4550 2950
-	1    0    0    -1
-$EndComp
-Wire Wire Line
-	4550 2800 4550 2750
-Connection ~ 4550 2750
-Wire Wire Line
-	4550 3100 4550 3150
-Connection ~ 4550 3150
+P 4500 3000
+F 0 "R6" H 4550 3050 50  0000 L CNN
+F 1 "5.1k" H 4550 2950 50  0000 L CNN
+F 2 "Resistor_SMD:R_0603_1608Metric" V 4430 3000 50  0001 C CNN
+F 3 "~" H 4500 3000 50  0001 C CNN
+	1    4500 3000
+	1    0    0    -1
+$EndComp
 $Comp
 L Device:C C6
@@
 Text Label 7700 2000 0    50   ~ 0
 +5v
-Text Label 7000 2650 0    50   ~ 0
+Text Label 7200 2650 0    50   ~ 0
 Out
 Text Label 6850 3000 0    50   ~ 0
 Select
-Text Label 4550 2750 0    50   ~ 0
+Text Label 4400 2350 0    50   ~ 0
 In
+Connection ~ 4500 3150
+Wire Wire Line
+	4500 2850 4500 2750
+Connection ~ 4500 2750
+Wire Wire Line
+	4500 2750 4550 2750
+Wire Wire Line
+	3500 2350 4500 2350
+Wire Wire Line
+	4500 2350 4500 2750
+$Comp
+L Amp-rescue:Conn-My_Library J7
+U 1 1 63D437C1
+P 3400 2750
+F 0 "J7" H 3428 2796 50  0001 L CNN
+F 1 "Conn" H 3428 2705 50  0001 L CNN
+F 2 "My-library:SMD-CONN" H 3450 2600 50  0001 C CNN
+F 3 "~" H 3400 2750 50  0001 C CNN
+	1    3400 2750
+	-1   0    0    1
+$EndComp
+Wire Wire Line
+	6350 3000 6350 3450
+Wire Wire Line
+	6350 3450 4350 3450
+Connection ~ 6350 3000
+Wire Wire Line
+	5100 2850 5250 2850
+Connection ~ 5100 3150
+Wire Wire Line
+	5100 3150 5250 3150
+Wire Wire Line
+	4500 3150 5100 3150
+Text Label 5700 1800 0    50   ~ 0
+3.3v
+Wire Wire Line
+	6800 2000 6800 1800
+Wire Wire Line
+	3500 3150 3950 3150
+$Comp
+L My_Library:TS5A3167DBVR U4
+U 1 1 63D0B70A
+P 4050 2750
+F 0 "U4" H 3950 2900 50  0000 L CNN
+F 1 "TS5A3167DBVR" H 3850 2200 50  0000 L CNN
+F 2 "Package_TO_SOT_SMD:SOT-23-5" H 3815 2495 50  0001 C CNN
+F 3 " http://www.ti.com/lit/ds/symlink/ts5a3166.pdf" H 4050 2850 50  0001 C CNN
+	1    4050 2750
+	-1   0    0    -1
+$EndComp
+Wire Wire Line
+	4350 2850 4350 3450
+Wire Wire Line
+	3950 2450 3950 1800
+Wire Wire Line
+	4350 2750 4500 2750
+Wire Wire Line
+	3950 1800 6800 1800
+Wire Wire Line
+	3950 3050 3950 3150
+Connection ~ 3950 3150
+Wire Wire Line
+	3950 3150 4500 3150
+Wire Wire Line
+	6300 2650 6600 2650
+Wire Wire Line
+	7200 2650 7300 2650
+Wire Wire Line
+	7200 2750 7200 3000
+Wire Wire Line
+	6350 3000 7200 3000
+Wire Wire Line
+	7200 3000 7300 3000
+Connection ~ 7200 3000
+Text Label 3500 2750 0    50   ~ 0
+Signal
+Wire Wire Line
+	3500 2750 3750 2750
 $EndSCHEMATC

Commit message: изменено:      kicad/Amp/Amp-cache.lib 	изменено:      kicad/Amp/Amp.kicad_pcb 	изменено:      kicad/Amp/Amp.kicad_pcb-bak 	изменено:      kicad/Amp/Amp.sch 	изменено:      kicad/Amp/Amp.sch-bak 	изменено:      kicad/Amp/fp-info-cache
Parts:
- removed J1, J2: Conn, My-library:connBig, symbol Amp-rescue:Conn-My_Library
- added L1: 47uH, Inductor_SMD:L_0805_2012Metric, symbol Device:L
- added Z1: MCUSD18A40B12RS, My-library:MCUSD18A40B12RS, symbol My_Library:MCUSD18A40B12RS
- C3: value 1uF -> 10n
- J3, J4, J5, J6, J7: symbol Amp-rescue:Conn-My_Library -> Amp-rescue:Conn-My_Library-Amp-rescue
- R2, R3: value 100k -> 20k
- U4: symbol My_Library:TS5A3167DBVR -> Amp-rescue:TS5A3167DBVR-My_Library
Connections:
- wire segments 51 -> 50
Other:
- moved on the sheet: C3
Changed lines of the file:
@@
 $EndDescr
-$Comp
-L Amp-rescue:Conn-My_Library J1
-U 1 1 63C7E189
-P 3400 2350
-F 0 "J1" H 3342 2165 50  0001 C CNN
-F 1 "Conn" H 3342 2256 50  0001 C CNN
-F 2 "My-library:connBig" H 3450 2200 50  0001 C CNN
-F 3 "~" H 3400 2350 50  0001 C CNN
-	1    3400 2350
-	-1   0    0    1
-$EndComp
 $Comp
 L Device:C C2
@@
 $EndComp
 $Comp
-L power:GND #PWR02
-U 1 1 63C7F0B0
-P 5250 3250
-F 0 "#PWR02" H 5250 3000 50  0001 C CNN
-F 1 "GND" H 5255 3077 50  0001 C CNN
-F 2 "" H 5250 3250 50  0001 C CNN
-F 3 "" H 5250 3250 50  0001 C CNN
-	1    5250 3250
-	1    0    0    -1
-$EndComp
-$Comp
-L Amp-rescue:Conn-My_Library J2
-U 1 1 63C7FD46
-P 3400 3150
-F 0 "J2" H 3342 2965 50  0001 C CNN
-F 1 "Conn" H 3342 3056 50  0001 C CNN
-F 2 "My-library:connBig" H 3450 3000 50  0001 C CNN
-F 3 "~" H 3400 3150 50  0001 C CNN
-	1    3400 3150
-	-1   0    0    1
-$EndComp
-$Comp
-L Amp-rescue:Conn-My_Library J6
+L Amp-rescue:Conn-My_Library-Amp-rescue J6
 U 1 1 63C80349
 P 7400 3150
@@
 U 1 1 63C8294F
 P 5250 3000
-F 0 "R3" H 5050 2800 50  0000 L CNN
-F 1 "100k" H 5000 2700 50  0000 L CNN
+F 0 "R3" H 5300 2800 50  0000 L CNN
+F 1 "20k" H 5300 2700 50  0000 L CNN
 F 2 "Resistor_SMD:R_0603_1608Metric" V 5180 3000 50  0001 C CNN
 F 3 "~" H 5250 3000 50  0001 C CNN
@@
 L Device:C C3
 U 1 1 63C8351B
-P 5100 3000
+P 5050 3000
 F 0 "C3" H 4850 3050 50  0000 L CNN
-F 1 "1uF" H 4850 2950 50  0000 L CNN
-F 2 "Capacitor_SMD:C_0603_1608Metric" H 5138 2850 50  0001 C CNN
-F 3 "~" H 5100 3000 50  0001 C CNN
-	1    5100 3000
+F 1 "10n" H 4800 2950 50  0000 L CNN
+F 2 "Capacitor_SMD:C_0603_1608Metric" H 5088 2850 50  0001 C CNN
+F 3 "~" H 5050 3000 50  0001 C CNN
+	1    5050 3000
 	1    0    0    -1
 $EndComp
@@
 	5250 2550 5250 2850
 Connection ~ 5250 2850
-Wire Wire Line
-	5250 3150 5250 3250
 Connection ~ 5250 3150
 Wire Wire Line
@@
 U 1 1 63C8A2D1
 P 6350 2100
-F 0 "Q1" V 6587 2100 50  0000 C CNN
+F 0 "Q1" V 6450 2100 50  0000 C CNN
 F 1 "Q_NPN_BEC" V 6587 2100 50  0001 C CNN
 F 2 "Package_TO_SOT_SMD:SOT-23" H 6550 2200 50  0001 C CNN
@@
 $EndComp
 $Comp
-L Amp-rescue:Conn-My_Library J3
+L Amp-rescue:Conn-My_Library-Amp-rescue J3
 U 1 1 63C8F41C
-P 7850 2000
-F 0 "J3" H 7878 2046 50  0001 L CNN
-F 1 "Conn" H 7878 1955 50  0001 L CNN
-F 2 "My-library:SMD-CONN" H 7900 1850 50  0001 C CNN
-F 3 "~" H 7850 2000 50  0001 C CNN
-	1    7850 2000
-	1    0    0    -1
-$EndComp
-$Comp
-L Amp-rescue:Conn-My_Library J5
+P 8100 2000
+F 0 "J3" H 8128 2046 50  0001 L CNN
+F 1 "Conn" H 8128 1955 50  0001 L CNN
+F 2 "My-library:SMD-CONN" H 8150 1850 50  0001 C CNN
+F 3 "~" H 8100 2000 50  0001 C CNN
+	1    8100 2000
+	1    0    0    -1
+$EndComp
+$Comp
+L Amp-rescue:Conn-My_Library-Amp-rescue J5
 U 1 1 63C8F7BE
 P 7400 2650
@@
 $EndComp
 $Comp
-L Amp-rescue:Conn-My_Library J4
+L Amp-rescue:Conn-My_Library-Amp-rescue J4
 U 1 1 63C92E60
-P 7400 3000
-F 0 "J4" H 7428 3046 50  0001 L CNN
-F 1 "Conn" H 7428 2955 50  0001 L CNN
-F 2 "My-library:SMD-CONN" H 7450 2850 50  0001 C CNN
-F 3 "~" H 7400 3000 50  0001 C CNN
-	1    7400 3000
+P 7400 3450
+F 0 "J4" H 7428 3496 50  0001 L CNN
+F 1 "Conn" H 7428 3405 50  0001 L CNN
+F 2 "My-library:SMD-CONN" H 7450 3300 50  0001 C CNN
+F 3 "~" H 7400 3450 50  0001 C CNN
+	1    7400 3450
 	1    0    0    -1
 $EndComp
@@
 P 5250 2150
 F 0 "R2" H 5320 2196 50  0000 L CNN
-F 1 "100k" H 5320 2105 50  0000 L CNN
+F 1 "20k" H 5320 2105 50  0000 L CNN
 F 2 "Resistor_SMD:R_0603_1608Metric" V 5180 2150 50  0001 C CNN
 F 3 "~" H 5250 2150 50  0001 C CNN
@@
 P 6900 2650
 F 0 "U2" H 6800 2800 50  0000 L CNN
-F 1 "TS5A3166DBVR" H 6650 2050 50  0000 L CNN
+F 1 "TS5A3166DBVR" H 6650 2050 50  0001 L CNN
 F 2 "Package_TO_SOT_SMD:SOT-23-5" H 6850 2500 50  0001 C CNN
 F 3 " http://www.ti.com/lit/ds/symlink/ts5a3166.pdf" H 6900 2750 50  0001 C CNN
@@
 	-1   0    0    -1
 $EndComp
-Wire Wire Line
-	6350 2600 6350 2750
-Wire Wire Line
-	6350 2750 6400 2750
-Wire Wire Line
-	6350 2750 6350 3000
-Connection ~ 6350 2750
 Wire Wire Line
 	6800 2950 6800 3150
@@
 Wire Wire Line
 	7650 2000 7700 2000
-Connection ~ 7700 2000
-Wire Wire Line
-	7700 2000 7750 2000
 Wire Wire Line
 	6950 2000 7050 2000
@@
 Wire Wire Line
 	6000 2000 6150 2000
-Text Label 7700 2000 0    50   ~ 0
+Text Label 8000 2000 0    50   ~ 0
 +5v
 Text Label 7200 2650 0    50   ~ 0
 Out
-Text Label 6850 3000 0    50   ~ 0
+Text Label 7200 3400 0    50   ~ 0
 Select
 Text Label 4400 2350 0    50   ~ 0
@@
 	4500 2750 4550 2750
 Wire Wire Line
-	3500 2350 4500 2350
-Wire Wire Line
 	4500 2350 4500 2750
 $Comp
-L Amp-rescue:Conn-My_Library J7
+L Amp-rescue:Conn-My_Library-Amp-rescue J7
 U 1 1 63D437C1
-P 3400 2750
-F 0 "J7" H 3428 2796 50  0001 L CNN
-F 1 "Conn" H 3428 2705 50  0001 L CNN
-F 2 "My-library:SMD-CONN" H 3450 2600 50  0001 C CNN
-F 3 "~" H 3400 2750 50  0001 C CNN
-	1    3400 2750
+P 3500 2150
+F 0 "J7" H 3528 2196 50  0001 L CNN
+F 1 "Conn" H 3528 2105 50  0001 L CNN
+F 2 "My-library:SMD-CONN" H 3550 2000 50  0001 C CNN
+F 3 "~" H 3500 2150 50  0001 C CNN
+	1    3500 2150
 	-1   0    0    1
 $EndComp
 Wire Wire Line
-	6350 3000 6350 3450
-Wire Wire Line
 	6350 3450 4350 3450
-Connection ~ 6350 3000
-Wire Wire Line
-	5100 2850 5250 2850
-Connection ~ 5100 3150
-Wire Wire Line
-	5100 3150 5250 3150
-Wire Wire Line
-	4500 3150 5100 3150
-Text Label 5700 1800 0    50   ~ 0
+Wire Wire Line
+	4500 3150 5050 3150
+Text Label 5700 1850 0    50   ~ 0
 3.3v
 Wire Wire Line
-	6800 2000 6800 1800
-Wire Wire Line
-	3500 3150 3950 3150
-$Comp
-L My_Library:TS5A3167DBVR U4
+	6800 2000 6800 1850
+$Comp
+L Amp-rescue:TS5A3167DBVR-My_Library U4
 U 1 1 63D0B70A
 P 4050 2750
 F 0 "U4" H 3950 2900 50  0000 L CNN
-F 1 "TS5A3167DBVR" H 3850 2200 50  0000 L CNN
+F 1 "TS5A3167DBVR" H 3850 2250 50  0001 L CNN
 F 2 "Package_TO_SOT_SMD:SOT-23-5" H 3815 2495 50  0001 C CNN
 F 3 " http://www.ti.com/lit/ds/symlink/ts5a3166.pdf" H 4050 2850 50  0001 C CNN
@@
 	4350 2850 4350 3450
 Wire Wire Line
-	3950 2450 3950 1800
+	3950 2450 3950 1850
 Wire Wire Line
 	4350 2750 4500 2750
-Wire Wire Line
-	3950 1800 6800 1800
 Wire Wire Line
 	3950 3050 3950 3150
@@
 Wire Wire Line
 	7200 2650 7300 2650
-Wire Wire Line
-	7200 2750 7200 3000
-Wire Wire Line
-	6350 3000 7200 3000
-Wire Wire Line
-	7200 3000 7300 3000
-Connection ~ 7200 3000
-Text Label 3500 2750 0    50   ~ 0
+Text Label 3600 2150 0    50   ~ 0
 Signal
-Wire Wire Line
-	3500 2750 3750 2750
+$Comp
+L power:GND #PWR02
+U 1 1 63CE834D
+P 5600 3250
+F 0 "#PWR02" H 5600 3000 50  0001 C CNN
+F 1 "GND" H 5605 3077 50  0001 C CNN
+F 2 "" H 5600 3250 50  0001 C CNN
+F 3 "" H 5600 3250 50  0001 C CNN
+	1    5600 3250
+	1    0    0    -1
+$EndComp
+Wire Wire Line
+	5600 3150 5600 3250
+$Comp
+L Device:L L1
+U 1 1 63CECB33
+P 7850 2000
+F 0 "L1" V 8040 2000 50  0000 C CNN
+F 1 "47uH" V 7949 2000 50  0000 C CNN
+F 2 "Inductor_SMD:L_0805_2012Metric" H 7850 2000 50  0001 C CNN
+F 3 "~" H 7850 2000 50  0001 C CNN
+	1    7850 2000
+	0    -1   -1   0
+$EndComp
+Connection ~ 7700 2000
+Connection ~ 5050 3150
+Wire Wire Line
+	5050 2850 5250 2850
+Wire Wire Line
+	5050 3150 5250 3150
+Wire Wire Line
+	3950 1850 6800 1850
+Wire Wire Line
+	7200 3450 6350 3450
+Connection ~ 6350 3450
+Wire Wire Line
+	6350 2600 6350 3450
+Wire Wire Line
+	7200 2750 7200 3450
+Wire Wire Line
+	7300 3450 7200 3450
+Connection ~ 7200 3450
+$Comp
+L My_Library:MCUSD18A40B12RS Z1
+U 1 1 63D25829
+P 3550 2750
+F 0 "Z1" H 3550 2650 50  0000 L CNN
+F 1 "MCUSD18A40B12RS" H 2700 2600 50  0001 L CNN
+F 2 "My-library:MCUSD18A40B12RS" H 3550 2750 50  0001 C CNN
+F 3 "" H 3550 2750 50  0001 C CNN
+	1    3550 2750
+	1    0    0    -1
+$EndComp
+Wire Wire Line
+	3750 2750 3750 2150
+Wire Wire Line
+	3750 2150 3600 2150
+Wire Wire Line
+	3550 2550 3550 2350
+Wire Wire Line
+	3550 2350 4500 2350
+Wire Wire Line
+	3550 2950 3550 3150
+Wire Wire Line
+	3550 3150 3950 3150
 $EndSCHEMATC

Commit message: изменено:      kicad/Amp/Amp-cache.lib 	изменено:      kicad/Amp/Amp.sch 	изменено:      kicad/Amp/Amp.sch-bak
Parts:
- J3, J4, J5, J6, J7: symbol Amp-rescue:Conn-My_Library-Amp-rescue -> Amp-rescue:Conn-My_Library-Amp-rescue-Amp-rescue
- U4: symbol Amp-rescue:TS5A3167DBVR-My_Library -> Amp-rescue:TS5A3167DBVR-My_Library-Amp-rescue
- Z1: symbol My_Library:MCUSD18A40B12RS -> Amp-rescue:MCUSD18A40B12RS-My_Library
Changed lines of the file:
@@
 $EndComp
 $Comp
-L Amp-rescue:Conn-My_Library-Amp-rescue J6
+L Amp-rescue:Conn-My_Library-Amp-rescue-Amp-rescue J6
 U 1 1 63C80349
 P 7400 3150
@@
 $EndComp
 $Comp
-L Amp-rescue:Conn-My_Library-Amp-rescue J3
+L Amp-rescue:Conn-My_Library-Amp-rescue-Amp-rescue J3
 U 1 1 63C8F41C
 P 8100 2000
@@
 $EndComp
 $Comp
-L Amp-rescue:Conn-My_Library-Amp-rescue J5
+L Amp-rescue:Conn-My_Library-Amp-rescue-Amp-rescue J5
 U 1 1 63C8F7BE
 P 7400 2650
@@
 $EndComp
 $Comp
-L Amp-rescue:Conn-My_Library-Amp-rescue J4
+L Amp-rescue:Conn-My_Library-Amp-rescue-Amp-rescue J4
 U 1 1 63C92E60
 P 7400 3450
@@
 	4500 2350 4500 2750
 $Comp
-L Amp-rescue:Conn-My_Library-Amp-rescue J7
+L Amp-rescue:Conn-My_Library-Amp-rescue-Amp-rescue J7
 U 1 1 63D437C1
 P 3500 2150
@@
 	6800 2000 6800 1850
 $Comp
-L Amp-rescue:TS5A3167DBVR-My_Library U4
+L Amp-rescue:TS5A3167DBVR-My_Library-Amp-rescue U4
 U 1 1 63D0B70A
 P 4050 2750
@@
 Connection ~ 7200 3450
 $Comp
-L My_Library:MCUSD18A40B12RS Z1
+L Amp-rescue:MCUSD18A40B12RS-My_Library Z1
 U 1 1 63D25829
 P 3550 2750

Commit message: изменено:      kicad/Amp/Amp-cache.lib 	изменено:      kicad/Amp/Amp.kicad_pcb 	изменено:      kicad/Amp/Amp.kicad_pcb-bak 	изменено:      kicad/Amp/Amp.sch 	изменено:      kicad/Amp/Amp.sch-bak 	изменено:      kicad/Amp/fp-info-cache
Parts:
- removed Q1: Q_NPN_BEC, Package_TO_SOT_SMD:SOT-23, symbol Device:Q_NPN_BEC
- removed U1: AD8541, Package_TO_SOT_SMD:TSOT-23-5, symbol Amplifier_Operational:AD8603
- removed U4: TS5A3167DBVR, Package_TO_SOT_SMD:SOT-23-5, symbol Amp-rescue:TS5A3167DBVR-My_Library-Amp-rescue
- removed Z1: MCUSD18A40B12RS, My-library:MCUSD18A40B12RS, symbol Amp-rescue:MCUSD18A40B12RS-My_Library
- added C1: 10uF, Capacitor_SMD:C_0603_1608Metric, symbol Device:C
- added C6: 1.5n, Resistor_SMD:R_0402_1005Metric, symbol Device:C
- added C7: 0.1uF, Capacitor_SMD:C_0402_1005Metric, symbol Device:C
- added D1: MAX4477, Package_SO:MSOP-8_3x3mm_P0.65mm, symbol My_Library:MAX4477
- added D2: TLV3501, Package_TO_SOT_SMD:SOT-23-6, symbol My_Library:TLV3501-2
- added R1: 5.1k, Resistor_SMD:R_0402_1005Metric, symbol Device:R
- added R7, R9: 100k, Resistor_SMD:R_0402_1005Metric, symbol Device:R
- added R8: 10k, Resistor_SMD:R_0402_1005Metric, symbol Device:R
- added Z1: MCUSD18A40B12RS, My-library:MCUSD18A40B12RS, symbol My_Library:MCUSD18A40B12RS
- C2: renamed from C1; footprint Resistor_SMD:R_0603_1608Metric -> Resistor_SMD:R_0402_1005Metric
- C3: value 10n -> 0.1uF; footprint Capacitor_SMD:C_0603_1608Metric -> Capacitor_SMD:C_0402_1005Metric
- C4: value 10n -> 100n; footprint Resistor_SMD:R_0603_1608Metric -> Resistor_SMD:R_0402_1005Metric
- J1: renamed from J7; symbol Amp-rescue:Conn-My_Library-Amp-rescue-Amp-rescue -> Amp-rescue:Conn-My_Library-Amp-rescue-Amp-rescue-Amp-rescue
- J2: renamed from J5; symbol Amp-rescue:Conn-My_Library-Amp-rescue-Amp-rescue -> Amp-rescue:Conn-My_Library-Amp-rescue-Amp-rescue-Amp-rescue
- J3: renamed from J6; symbol Amp-rescue:Conn-My_Library-Amp-rescue-Amp-rescue -> Amp-rescue:Conn-My_Library-Amp-rescue-Amp-rescue-Amp-rescue
- J4: symbol Amp-rescue:Conn-My_Library-Amp-rescue-Amp-rescue -> Amp-rescue:Conn-My_Library-Amp-rescue-Amp-rescue-Amp-rescue
- J5: renamed from J3; symbol Amp-rescue:Conn-My_Library-Amp-rescue-Amp-rescue -> Amp-rescue:Conn-My_Library-Amp-rescue-Amp-rescue-Amp-rescue
- R10: renamed from R5; value 10k -> 5.1k; footprint Resistor_SMD:R_0603_1608Metric -> Resistor_SMD:R_0402_1005Metric
- R2: renamed from R1; value 5.1k -> 1k; footprint Resistor_SMD:R_0603_1608Metric -> Resistor_SMD:R_0402_1005Metric
- R3: renamed from R2; value 20k -> 100k; footprint Resistor_SMD:R_0603_1608Metric -> Resistor_SMD:R_0402_1005Metric
- R4: renamed from R3; value 20k -> 100k; footprint Resistor_SMD:R_0603_1608Metric -> Resistor_SMD:R_0402_1005Metric
- R5: renamed from R4; footprint Resistor_SMD:R_0603_1608Metric -> Resistor_SMD:R_0402_1005Metric
- R6: footprint Resistor_SMD:R_0603_1608Metric -> Resistor_SMD:R_0402_1005Metric
- renumbered C7 to C10, C2 to C5, C6 to C8, C5 to C9, U2 to U1, U3 to U2
Connections:
- net labels added: Sel, Sig
- net labels removed: Select, Signal
- wire segments 50 -> 70
Other:
- moved on the sheet: C10, C2, C3, C5, C8, C9, L1, R10, R2, R3, R4, R5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
