File: kicad/Amp/Amp.sch (KiCad schematic (older format))
At the start: 31 parts, among them J1 Conn, J2 Conn, J3 Conn, J4 Conn, J5 Conn, U1 TS5A3166DBVR, U2 MCP1700

Commit message: изменено:      kicad/Amp/Amp-cache.lib 	изменено:      kicad/Amp/Amp.sch 	изменено:      kicad/Amp/Amp.sch-bak
Parts:
- D1: symbol My_Library:MAX4477 -> Amp-rescue:MAX4477-My_Library
- D2: symbol My_Library:TLV3501-2 -> Amp-rescue:TLV3501-2-My_Library
- J1, J2, J3, J4, J5: symbol Amp-rescue:Conn-My_Library-Amp-rescue-Amp-rescue-Amp-rescue -> Amp-rescue:Conn-My_Library-Amp-rescue-Amp-rescue-Amp-rescue-Amp-rescue
- Z1: symbol My_Library:MCUSD18A40B12RS -> Amp-rescue:MCUSD18A40B12RS-My_Library
Changed lines of the file:
@@
 $EndComp
 $Comp
-L Amp-rescue:Conn-My_Library-Amp-rescue-Amp-rescue-Amp-rescue J3
+L Amp-rescue:Conn-My_Library-Amp-rescue-Amp-rescue-Amp-rescue-Amp-rescue J3
 U 1 1 63C80349
 P 8600 4650
@@
 $EndComp
 $Comp
-L Amp-rescue:Conn-My_Library-Amp-rescue-Amp-rescue-Amp-rescue J5
+L Amp-rescue:Conn-My_Library-Amp-rescue-Amp-rescue-Amp-rescue-Amp-rescue J5
 U 1 1 63C8F41C
 P 9150 3000
@@
 $EndComp
 $Comp
-L Amp-rescue:Conn-My_Library-Amp-rescue-Amp-rescue-Amp-rescue J4
+L Amp-rescue:Conn-My_Library-Amp-rescue-Amp-rescue-Amp-rescue-Amp-rescue J4
 U 1 1 63C92E60
 P 8600 4900
@@
 In
 $Comp
-L Amp-rescue:Conn-My_Library-Amp-rescue-Amp-rescue-Amp-rescue J1
+L Amp-rescue:Conn-My_Library-Amp-rescue-Amp-rescue-Amp-rescue-Amp-rescue J1
 U 1 1 63D437C1
 P 2950 3600
@@
 Connection ~ 8750 3000
 $Comp
-L My_Library:MAX4477 D1
+L Amp-rescue:MAX4477-My_Library D1
 U 1 1 63E14065
 P 5250 3750
@@
 $EndComp
 $Comp
-L My_Library:MAX4477 D1
+L Amp-rescue:MAX4477-My_Library D1
 U 2 1 63E14B3D
 P 6600 3900
@@
 $EndComp
 $Comp
-L My_Library:TLV3501-2 D2
+L Amp-rescue:TLV3501-2-My_Library D2
 U 1 1 63E15A52
 P 8050 4000
@@
 	3050 3600 3150 3600
 $Comp
-L Amp-rescue:Conn-My_Library-Amp-rescue-Amp-rescue-Amp-rescue J2
+L Amp-rescue:Conn-My_Library-Amp-rescue-Amp-rescue-Amp-rescue-Amp-rescue J2
 U 1 1 63C8F7BE
 P 8600 4000
@@
 Out
 $Comp
-L My_Library:MCUSD18A40B12RS Z1
+L Amp-rescue:MCUSD18A40B12RS-My_Library Z1
 U 1 1 640B9EB9
 P 4150 4200

Commit message: изменено:      kicad/Amp/Amp-cache.lib 	изменено:      kicad/Amp/Amp.kicad_pcb 	изменено:      kicad/Amp/Amp.kicad_pcb-bak 	изменено:      kicad/Amp/Amp.sch 	изменено:      kicad/Amp/Amp.sch-bak
Parts:
- C2, C4, C6: footprint Resistor_SMD:R_0402_1005Metric -> Capacitor_SMD:C_0402_1005Metric
- D1: symbol Amp-rescue:MAX4477-My_Library -> Amp-rescue:MAX4477-My_Library-Amp-rescue
- D2: symbol Amp-rescue:TLV3501-2-My_Library -> Amp-rescue:TLV3501-2-My_Library-Amp-rescue
- J1, J2, J3, J4, J5: symbol Amp-rescue:Conn-My_Library-Amp-rescue-Amp-rescue-Amp-rescue-Amp-rescue -> Amp-rescue:Conn-My_Library-Amp-rescue-Amp-rescue-Amp-rescue-Amp-rescue-Amp-rescue
- Z1: symbol Amp-rescue:MCUSD18A40B12RS-My_Library -> Amp-rescue:MCUSD18A40B12RS-My_Library-Amp-rescue
Connections:
- net In: now also C2.2, R1.1, U1.1, Z1.+
Changed lines of the file:
@@
 $EndComp
 $Comp
-L Amp-rescue:Conn-My_Library-Amp-rescue-Amp-rescue-Amp-rescue-Amp-rescue J3
+L Amp-rescue:Conn-My_Library-Amp-rescue-Amp-rescue-Amp-rescue-Amp-rescue-Amp-rescue J3
 U 1 1 63C80349
 P 8600 4650
@@
 F 0 "C2" V 4050 3600 50  0000 C CNN
 F 1 "1.5n" V 4150 3600 50  0000 C CNN
-F 2 "Resistor_SMD:R_0402_1005Metric" H 4338 3450 50  0001 C CNN
+F 2 "Capacitor_SMD:C_0402_1005Metric" H 4338 3450 50  0001 C CNN
 F 3 "~" H 4300 3600 50  0001 C CNN
 	1    4300 3600
@@
 $EndComp
 $Comp
-L Amp-rescue:Conn-My_Library-Amp-rescue-Amp-rescue-Amp-rescue-Amp-rescue J5
+L Amp-rescue:Conn-My_Library-Amp-rescue-Amp-rescue-Amp-rescue-Amp-rescue-Amp-rescue J5
 U 1 1 63C8F41C
 P 9150 3000
@@
 $EndComp
 $Comp
-L Amp-rescue:Conn-My_Library-Amp-rescue-Amp-rescue-Amp-rescue-Amp-rescue J4
+L Amp-rescue:Conn-My_Library-Amp-rescue-Amp-rescue-Amp-rescue-Amp-rescue-Amp-rescue J4
 U 1 1 63C92E60
 P 8600 4900
@@
 Text Label 8400 4900 0    50   ~ 0
 Sel
-Text Label 4000 3750 0    50   ~ 0
+Text Label 4000 3600 0    50   ~ 0
 In
 $Comp
-L Amp-rescue:Conn-My_Library-Amp-rescue-Amp-rescue-Amp-rescue-Amp-rescue J1
+L Amp-rescue:Conn-My_Library-Amp-rescue-Amp-rescue-Amp-rescue-Amp-rescue-Amp-rescue J1
 U 1 1 63D437C1
 P 2950 3600
@@
 Connection ~ 8750 3000
 $Comp
-L Amp-rescue:MAX4477-My_Library D1
+L Amp-rescue:MAX4477-My_Library-Amp-rescue D1
 U 1 1 63E14065
 P 5250 3750
@@
 $EndComp
 $Comp
-L Amp-rescue:MAX4477-My_Library D1
+L Amp-rescue:MAX4477-My_Library-Amp-rescue D1
 U 2 1 63E14B3D
 P 6600 3900
@@
 $EndComp
 $Comp
-L Amp-rescue:TLV3501-2-My_Library D2
+L Amp-rescue:TLV3501-2-My_Library-Amp-rescue D2
 U 1 1 63E15A52
 P 8050 4000
@@
 F 0 "C4" V 5500 3750 50  0000 C CNN
 F 1 "100n" V 5600 3750 50  0000 C CNN
-F 2 "Resistor_SMD:R_0402_1005Metric" H 5788 3600 50  0001 C CNN
+F 2 "Capacitor_SMD:C_0402_1005Metric" H 5788 3600 50  0001 C CNN
 F 3 "~" H 5750 3750 50  0001 C CNN
 	1    5750 3750
@@
 F 0 "C6" V 7250 3900 50  0000 C CNN
 F 1 "1.5n" V 7350 3900 50  0000 C CNN
-F 2 "Resistor_SMD:R_0402_1005Metric" H 7138 3750 50  0001 C CNN
+F 2 "Capacitor_SMD:C_0402_1005Metric" H 7138 3750 50  0001 C CNN
 F 3 "~" H 7100 3900 50  0001 C CNN
 	1    7100 3900
@@
 	3050 3600 3150 3600
 $Comp
-L Amp-rescue:Conn-My_Library-Amp-rescue-Amp-rescue-Amp-rescue-Amp-rescue J2
+L Amp-rescue:Conn-My_Library-Amp-rescue-Amp-rescue-Amp-rescue-Amp-rescue-Amp-rescue J2
 U 1 1 63C8F7BE
 P 8600 4000
@@
 Out
 $Comp
-L Amp-rescue:MCUSD18A40B12RS-My_Library Z1
+L Amp-rescue:MCUSD18A40B12RS-My_Library-Amp-rescue Z1
 U 1 1 640B9EB9
 P 4150 4200

Commit message: изменено:      kicad/Amp/Amp-cache.lib 	изменено:      kicad/Amp/Amp.sch 	изменено:      kicad/Amp/Amp.sch-bak
Parts:
- D1: symbol Amp-rescue:MAX4477-My_Library-Amp-rescue -> Amp-rescue:MAX4477-My_Library-Amp-rescue-Amp-rescue
- D2: symbol Amp-rescue:TLV3501-2-My_Library-Amp-rescue -> Amp-rescue:TLV3501-2-My_Library-Amp-rescue-Amp-rescue
- J1, J2, J3, J4, J5: symbol Amp-rescue:Conn-My_Library-Amp-rescue-Amp-rescue-Amp-rescue-Amp-rescue-Amp-rescue -> Amp-rescue:Conn-My_Library-Amp-rescue-Amp-rescue-Amp-rescue-Amp-rescue-Amp-rescue-Amp-rescue
- Z1: symbol Amp-rescue:MCUSD18A40B12RS-My_Library-Amp-rescue -> Amp-rescue:MCUSD18A40B12RS-My_Library-Amp-rescue-Amp-rescue
Changed lines of the file:
@@
 $EndComp
 $Comp
-L Amp-rescue:Conn-My_Library-Amp-rescue-Amp-rescue-Amp-rescue-Amp-rescue-Amp-rescue J3
+L Amp-rescue:Conn-My_Library-Amp-rescue-Amp-rescue-Amp-rescue-Amp-rescue-Amp-rescue-Amp-rescue J3
 U 1 1 63C80349
 P 8600 4650
@@
 $EndComp
 $Comp
-L Amp-rescue:Conn-My_Library-Amp-rescue-Amp-rescue-Amp-rescue-Amp-rescue-Amp-rescue J5
+L Amp-rescue:Conn-My_Library-Amp-rescue-Amp-rescue-Amp-rescue-Amp-rescue-Amp-rescue-Amp-rescue J5
 U 1 1 63C8F41C
 P 9150 3000
@@
 $EndComp
 $Comp
-L Amp-rescue:Conn-My_Library-Amp-rescue-Amp-rescue-Amp-rescue-Amp-rescue-Amp-rescue J4
+L Amp-rescue:Conn-My_Library-Amp-rescue-Amp-rescue-Amp-rescue-Amp-rescue-Amp-rescue-Amp-rescue J4
 U 1 1 63C92E60
 P 8600 4900
@@
 In
 $Comp
-L Amp-rescue:Conn-My_Library-Amp-rescue-Amp-rescue-Amp-rescue-Amp-rescue-Amp-rescue J1
+L Amp-rescue:Conn-My_Library-Amp-rescue-Amp-rescue-Amp-rescue-Amp-rescue-Amp-rescue-Amp-rescue J1
 U 1 1 63D437C1
 P 2950 3600
@@
 Connection ~ 8750 3000
 $Comp
-L Amp-rescue:MAX4477-My_Library-Amp-rescue D1
+L Amp-rescue:MAX4477-My_Library-Amp-rescue-Amp-rescue D1
 U 1 1 63E14065
 P 5250 3750
@@
 $EndComp
 $Comp
-L Amp-rescue:MAX4477-My_Library-Amp-rescue D1
+L Amp-rescue:MAX4477-My_Library-Amp-rescue-Amp-rescue D1
 U 2 1 63E14B3D
 P 6600 3900
@@
 $EndComp
 $Comp
-L Amp-rescue:TLV3501-2-My_Library-Amp-rescue D2
+L Amp-rescue:TLV3501-2-My_Library-Amp-rescue-Amp-rescue D2
 U 1 1 63E15A52
 P 8050 4000
@@
 	3050 3600 3150 3600
 $Comp
-L Amp-rescue:Conn-My_Library-Amp-rescue-Amp-rescue-Amp-rescue-Amp-rescue-Amp-rescue J2
+L Amp-rescue:Conn-My_Library-Amp-rescue-Amp-rescue-Amp-rescue-Amp-rescue-Amp-rescue-Amp-rescue J2
 U 1 1 63C8F7BE
 P 8600 4000
@@
 Out
 $Comp
-L Amp-rescue:MCUSD18A40B12RS-My_Library-Amp-rescue Z1
+L Amp-rescue:MCUSD18A40B12RS-My_Library-Amp-rescue-Amp-rescue Z1
 U 1 1 640B9EB9
 P 4150 4200

Commit message: изменено:      kicad/Amp/Amp-cache.lib 	изменено:      kicad/Amp/Amp.kicad_pcb 	изменено:      kicad/Amp/Amp.kicad_pcb-bak 	изменено:      kicad/Amp/Amp.sch 	изменено:      kicad/Amp/Amp.sch-bak
Parts:
- D1: symbol Amp-rescue:MAX4477-My_Library-Amp-rescue-Amp-rescue -> Amp-rescue:MAX4477-My_Library-Amp-rescue-Amp-rescue-Amp-rescue
- D2: symbol Amp-rescue:TLV3501-2-My_Library-Amp-rescue-Amp-rescue -> Amp-rescue:TLV3501-2-My_Library-Amp-rescue-Amp-rescue-Amp-rescue
- J1, J2, J3, J4, J5: symbol Amp-rescue:Conn-My_Library-Amp-rescue-Amp-rescue-Amp-rescue-Amp-rescue-Amp-rescue-Amp-rescue -> Amp-rescue:Conn-My_Library-Amp-rescue-Amp-rescue-Amp-rescue-Amp-rescue-Amp-rescue-Amp-rescue-Amp-rescue
- Z1: symbol Amp-rescue:MCUSD18A40B12RS-My_Library-Amp-rescue-Amp-rescue -> Amp-rescue:MCUSD18A40B12RS-My_Library-Amp-rescue-Amp-rescue-Amp-rescue
Changed lines of the file:
@@
 $EndComp
 $Comp
-L Amp-rescue:Conn-My_Library-Amp-rescue-Amp-rescue-Amp-rescue-Amp-rescue-Amp-rescue-Amp-rescue J3
+L Amp-rescue:Conn-My_Library-Amp-rescue-Amp-rescue-Amp-rescue-Amp-rescue-Amp-rescue-Amp-rescue-Amp-rescue J3
 U 1 1 63C80349
 P 8600 4650
@@
 $EndComp
 $Comp
-L Amp-rescue:Conn-My_Library-Amp-rescue-Amp-rescue-Amp-rescue-Amp-rescue-Amp-rescue-Amp-rescue J5
+L Amp-rescue:Conn-My_Library-Amp-rescue-Amp-rescue-Amp-rescue-Amp-rescue-Amp-rescue-Amp-rescue-Amp-rescue J5
 U 1 1 63C8F41C
 P 9150 3000
@@
 $EndComp
 $Comp
-L Amp-rescue:Conn-My_Library-Amp-rescue-Amp-rescue-Amp-rescue-Amp-rescue-Amp-rescue-Amp-rescue J4
+L Amp-rescue:Conn-My_Library-Amp-rescue-Amp-rescue-Amp-rescue-Amp-rescue-Amp-rescue-Amp-rescue-Amp-rescue J4
 U 1 1 63C92E60
 P 8600 4900
@@
 In
 $Comp
-L Amp-rescue:Conn-My_Library-Amp-rescue-Amp-rescue-Amp-rescue-Amp-rescue-Amp-rescue-Amp-rescue J1
+L Amp-rescue:Conn-My_Library-Amp-rescue-Amp-rescue-Amp-rescue-Amp-rescue-Amp-rescue-Amp-rescue-Amp-rescue J1
 U 1 1 63D437C1
 P 2950 3600
@@
 Connection ~ 8750 3000
 $Comp
-L Amp-rescue:MAX4477-My_Library-Amp-rescue-Amp-rescue D1
+L Amp-rescue:MAX4477-My_Library-Amp-rescue-Amp-rescue-Amp-rescue D1
 U 1 1 63E14065
 P 5250 3750
@@
 $EndComp
 $Comp
-L Amp-rescue:MAX4477-My_Library-Amp-rescue-Amp-rescue D1
+L Amp-rescue:MAX4477-My_Library-Amp-rescue-Amp-rescue-Amp-rescue D1
 U 2 1 63E14B3D
 P 6600 3900
@@
 $EndComp
 $Comp
-L Amp-rescue:TLV3501-2-My_Library-Amp-rescue-Amp-rescue D2
+L Amp-rescue:TLV3501-2-My_Library-Amp-rescue-Amp-rescue-Amp-rescue D2
 U 1 1 63E15A52
 P 8050 4000
@@
 	3050 3600 3150 3600
 $Comp
-L Amp-rescue:Conn-My_Library-Amp-rescue-Amp-rescue-Amp-rescue-Amp-rescue-Amp-rescue-Amp-rescue J2
+L Amp-rescue:Conn-My_Library-Amp-rescue-Amp-rescue-Amp-rescue-Amp-rescue-Amp-rescue-Amp-rescue-Amp-rescue J2
 U 1 1 63C8F7BE
 P 8600 4000
@@
 Out
 $Comp
-L Amp-rescue:MCUSD18A40B12RS-My_Library-Amp-rescue-Amp-rescue Z1
+L Amp-rescue:MCUSD18A40B12RS-My_Library-Amp-rescue-Amp-rescue-Amp-rescue Z1
 U 1 1 640B9EB9
 P 4150 4200
