File: kicad/Amp/Amp.kicad_pcb (KiCad board)
At the start: 2 copper layers, 30 x 25.6 mm, 31 parts, among them J1 Conn, J2 Conn, J3 Conn, J4 Conn, J5 Conn, U1 TS5A3166DBVR, U2 MCP1700

Commit message: изменено:      kicad/Amp/Amp-rescue.lib 	изменено:      kicad/Amp/Amp.kicad_pcb 	изменено:      stm32cubeide/Anemometer_G474CBT6_MATLAB/.settings/language.settings.xml
Parts:
- moved J5 21.1 mm to (45.6, 70.2)
- moved L1 18.8 mm to (43.2, 69.4), turned to 0 degrees
- moved C10 17.0 mm to (37.9, 66.1), turned to 90 degrees
- moved U2 14.1 mm to (40.2, 66.8), turned to -90 degrees
- moved J3 14.1 mm to (53.5, 66.8)
- moved C5 7.73 mm to (38.9, 63.7), turned to 180 degrees
- moved C1 2.65 mm to (46.6, 65.1)
- moved J1 1.99 mm to (55.6, 63.3)
- moved J4 1.84 mm to (48.3, 65.9)
- moved R2 1.84 mm to (48.0, 55.5)
- moved C2 1.84 mm to (50.0, 55.5)
- moved C3 1.84 mm to (49.1, 59.2)
- moved R5 1.84 mm to (46.0, 55.5)
- moved C9 1.84 mm to (49.3, 61.2)
- moved R7 1.84 mm to (46.2, 63.1)
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Routing:
- net GND: track 27.6 -> 11.4 mm, vias 4 -> 5
- net /3.3v: track 33.8 -> 24.3 mm
- net Net-(C10-Pad1): track 3.85 -> 5.25 mm
- net /+5v: track 2.48 -> 1.68 mm
- net /In: track 8.15 -> 7.41 mm
Other:
- net class Default removed
