File: kicad/Inv/invertor/invertor.sch (KiCad schematic (older format))
At the start: 24 parts, among them J1 Conn, J3 Conn, J4 Conn, J5 Conn, J6 Conn, Q1 IRF7343PBF, Q2 IRF7343PBF, Q3 IRLML6344

Commit message: изменено:      kicad/Inv/invertor/invertor-cache.lib 	изменено:      kicad/Inv/invertor/invertor.kicad_pcb 	изменено:      kicad/Inv/invertor/invertor.kicad_pcb-bak 	изменено:      kicad/Inv/invertor/invertor.sch 	изменено:      kicad/Inv/invertor/invertor.sch-bak 	изменено:      stm32cubeide/Anemometr_v3/Core/Inc/main.h 	изменено:      stm32cubeide/Anemometr_v3/Core/Src/main.c 	изменено:      stm32cubeide/Anemometr_v3/Release/Anemometr_3.bin 	изменено:      stm32cubeide/Anemometr_v3/Release/Anemometr_3.elf 	изменено:      stm32cubeide/Anemometr_v3/Release/Anemometr_3.hex 	изменено:      stm32cubeide/Anemometr_v3/Release/Anemometr_3.list 	изменено:      stm32cubeide/Anemometr_v3/Release/Core/Src/main.o 	изменено:      stm32cubeide/Anemometr_v3/Release/Core/Src/main.su
Parts:
- J1, J3, J4, J5, J6: symbol My_Library:Conn -> invertor-rescue:Conn-My_Library
Changed lines of the file:
@@
 $EndComp
 $Comp
-L My_Library:Conn J4
+L invertor-rescue:Conn-My_Library J4
 U 1 1 645979CD
 P 5800 1150
@@
 Connection ~ 5700 1150
 $Comp
-L My_Library:Conn J5
+L invertor-rescue:Conn-My_Library J5
 U 1 1 6459E72C
 P 6000 2050
@@
 $EndComp
 $Comp
-L My_Library:Conn J1
+L invertor-rescue:Conn-My_Library J1
 U 1 1 6459EF77
 P 4100 2050
@@
 $EndComp
 $Comp
-L My_Library:Conn J3
+L invertor-rescue:Conn-My_Library J3
 U 1 1 645A03DA
 P 3250 2750
@@
 $EndComp
 $Comp
-L My_Library:Conn J6
+L invertor-rescue:Conn-My_Library J6
 U 1 1 645A527F
 P 5800 3150

Commit message: изменено:      kicad/Inv/invertor/invertor.kicad_pcb 	изменено:      kicad/Inv/invertor/invertor.kicad_pcb-bak 	изменено:      kicad/Inv/invertor/invertor.sch 	изменено:      kicad/Inv/invertor/invertor.sch-bak 	изменено:      stm32cubeide/Anemometr_v3/.settings/language.settings.xml 	изменено:      stm32cubeide/Anemometr_v3/Core/Inc/main.h 	изменено:      stm32cubeide/Anemometr_v3/Core/Src/main.c 	изменено:      stm32cubeide/Anemometr_v3/Core/Src/stm32f1xx_it.c 	изменено:      stm32cubeide/Anemometr_v3/Release/Anemometr_3.bin 	изменено:      stm32cubeide/Anemometr_v3/Release/Anemometr_3.elf 	изменено:      stm32cubeide/Anemometr_v3/Release/Anemometr_3.hex 	изменено:      stm32cubeide/Anemometr_v3/Release/Anemometr_3.list 	изменено:      stm32cubeide/Anemometr_v3/Release/Anemometr_3.map 	изменено:      stm32cubeide/Anemometr_v3/Release/Core/Src/main.o 	изменено:      stm32cubeide/Anemometr_v3/Release/Core/Src/main.su 	изменено:      stm32cubeide/Anemometr_v3/Release/Core/Src/stm32f1xx_it.o
Parts:
- C1, C2, C3, C4: value 1nF -> 82nF
Changed lines of the file:
@@
 P 4700 1950
 F 0 "C1" H 4815 1996 50  0000 L CNN
-F 1 "1nF" H 4815 1905 50  0000 L CNN
+F 1 "82nF" H 4815 1905 50  0000 L CNN
 F 2 "Capacitor_SMD:C_0603_1608Metric" H 4738 1800 50  0001 C CNN
 F 3 "~" H 4700 1950 50  0001 C CNN
@@
 P 4700 2600
 F 0 "C2" H 4850 2700 50  0000 L CNN
-F 1 "1nF" H 4850 2600 50  0000 L CNN
+F 1 "82nF" H 4850 2600 50  0000 L CNN
 F 2 "Capacitor_SMD:C_0603_1608Metric" H 4738 2450 50  0001 C CNN
 F 3 "~" H 4700 2600 50  0001 C CNN
@@
 P 5400 2600
 F 0 "C4" H 5150 2700 50  0000 L CNN
-F 1 "1nF" H 5150 2600 50  0000 L CNN
+F 1 "82nF" H 5100 2600 50  0000 L CNN
 F 2 "Capacitor_SMD:C_0603_1608Metric" H 5438 2450 50  0001 C CNN
 F 3 "~" H 5400 2600 50  0001 C CNN
@@
 P 5400 1950
 F 0 "C3" H 5150 2000 50  0000 L CNN
-F 1 "1nF" H 5150 1900 50  0000 L CNN
+F 1 "82nF" H 5100 1900 50  0000 L CNN
 F 2 "Capacitor_SMD:C_0603_1608Metric" H 5438 1800 50  0001 C CNN
 F 3 "~" H 5400 1950 50  0001 C CNN
