File: kicad/Amp200/Amp200.sch (KiCad schematic (older format))
At the start: 44 parts, among them J1 Conn, J10 Conn, J2 Conn, J3 Conn, J4 Conn, J5 Conn, J6 Conn, J7 Conn, J8 Conn, J9 Conn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

Commit message: изменено:      kicad/Amp200/Amp200-cache.lib 	изменено:      kicad/Amp200/Amp200.kicad_pcb 	изменено:      kicad/Amp200/Amp200.sch 	изменено:      kicad/Amp200/Amp200.sch-bak 	изменено:      stm32cubeide/Anemometr_v3/Core/Src/main.c 	изменено:      stm32cubeide/Anemometr_v3/Core/Src/stm32f1xx_it.c 	изменено:      stm32cubeide/Anemometr_v3/Release/Anemometr_3.bin 	изменено:      stm32cubeide/Anemometr_v3/Release/Anemometr_3.elf 	изменено:      stm32cubeide/Anemometr_v3/Release/Anemometr_3.hex 	изменено:      stm32cubeide/Anemometr_v3/Release/Anemometr_3.list 	изменено:      stm32cubeide/Anemometr_v3/Release/Core/Src/main.o
Parts:
- D1: symbol My_Library:MAX4477 -> Amp200-rescue:MAX4477-My_Library
- D2: symbol My_Library:X9C103 -> Amp200-rescue:X9C103-My_Library
- D3: symbol My_Library:TLV3501-2 -> Amp200-rescue:TLV3501-2-My_Library
- D5: symbol My_Library:TS5A4595 -> Amp200-rescue:TS5A4595-My_Library
- J1, J10, J2, J3, J4, J5, J6, J7, J8, J9: symbol My_Library:Conn -> Amp200-rescue:Conn-My_Library
Changed lines of the file:
@@
 $EndDescr
 $Comp
-L My_Library:MAX4477 D1
+L Amp200-rescue:MAX4477-My_Library D1
 U 1 1 64214348
 P 4200 3000
@@
 $EndComp
 $Comp
-L My_Library:MAX4477 D1
+L Amp200-rescue:MAX4477-My_Library D1
 U 2 1 64214619
 P 6300 3650
@@
 $EndComp
 $Comp
-L My_Library:Conn J7
+L Amp200-rescue:Conn-My_Library J7
 U 1 1 64215621
 P 8500 4500
@@
 $EndComp
 $Comp
-L My_Library:X9C103 D2
+L Amp200-rescue:X9C103-My_Library D2
 U 1 1 64223D95
 P 4850 3300
@@
 Connection ~ 4850 3600
 $Comp
-L My_Library:TLV3501-2 D3
+L Amp200-rescue:TLV3501-2-My_Library D3
 U 1 1 64231BA0
 P 7750 3750
@@
 $EndComp
 $Comp
-L My_Library:Conn J6
+L Amp200-rescue:Conn-My_Library J6
 U 1 1 6426C541
 P 8500 3750
@@
 $EndComp
 $Comp
-L My_Library:Conn J8
+L Amp200-rescue:Conn-My_Library J8
 U 1 1 6426CAB6
 P 8500 4250
@@
 $EndComp
 $Comp
-L My_Library:Conn J9
+L Amp200-rescue:Conn-My_Library J9
 U 1 1 6426D093
 P 7350 1750
@@
 $EndComp
 $Comp
-L My_Library:Conn J2
+L Amp200-rescue:Conn-My_Library J2
 U 1 1 6426D58E
 P 4350 3200
@@
 $EndComp
 $Comp
-L My_Library:Conn J3
+L Amp200-rescue:Conn-My_Library J3
 U 1 1 6426DCFC
 P 4350 3300
@@
 $EndComp
 $Comp
-L My_Library:Conn J4
+L Amp200-rescue:Conn-My_Library J4
 U 1 1 6426E453
 P 4350 3400
@@
 $EndComp
 $Comp
-L My_Library:Conn J1
+L Amp200-rescue:Conn-My_Library J1
 U 1 1 6426E9F0
 P 2450 2850
@@
 $EndComp
 $Comp
-L My_Library:Conn J5
+L Amp200-rescue:Conn-My_Library J5
 U 1 1 642CF5AB
 P 8500 3300
@@
 	8100 4250 8400 4250
 $Comp
-L My_Library:TS5A4595 D5
+L Amp200-rescue:TS5A4595-My_Library D5
 U 1 1 643F68CC
 P 3250 3050
@@
 	4450 1450 6900 1450
 $Comp
-L My_Library:Conn J10
+L Amp200-rescue:Conn-My_Library J10
 U 1 1 64445C9E
 P 2450 4250

Commit message: изменено:      kicad/Amp200/Amp200.kicad_pcb 	изменено:      kicad/Amp200/Amp200.kicad_pcb-bak 	изменено:      kicad/Amp200/Amp200.sch 	изменено:      kicad/Amp200/Amp200.sch-bak 	изменено:      kicad/Amp200/fp-info-cache 	изменено:      stm32cubeide/Anemometr_v3/Core/Inc/main.h 	изменено:      stm32cubeide/Anemometr_v3/Release/Anemometr_3.bin 	изменено:      stm32cubeide/Anemometr_v3/Release/Anemometr_3.elf 	изменено:      stm32cubeide/Anemometr_v3/Release/Anemometr_3.hex 	изменено:      stm32cubeide/Anemometr_v3/Release/Anemometr_3.list 	изменено:      stm32cubeide/Anemometr_v3/Release/Anemometr_3.map 	изменено:      stm32cubeide/Anemometr_v3/Release/Core/Src/main.o 	изменено:      stm32cubeide/Anemometr_v3/Release/Core/Src/main.su
Parts:
- D1: footprint Package_SO:TSSOP-8_4.4x3mm_P0.65mm -> Package_SO:MSOP-8_3x3mm_P0.65mm
Connections:
- net +3.3v: now also U2.2 (VO); no longer U2.3 (VI)
- net +5v: now also U1.2 (VO); no longer U1.3 (VI)
- net at R1.2: now also D5.1 (Com); no longer D5.2 (Nc)
- net at C1.1: now also D5.2 (Nc); no longer D5.1 (Com)
- net at C7.1, L2.1: now also U2.3 (VI); no longer U2.2 (VO)
- net at C11.1, L1.1: now also U1.3 (VI); no longer U1.2 (VO)
Changed lines of the file:
@@
 F 0 "D1" H 4000 3100 50  0000 L CNN
 F 1 "MAX4477" H 4000 3000 50  0000 L CNN
-F 2 "Package_SO:TSSOP-8_4.4x3mm_P0.65mm" H 4200 3000 50  0001 C CNN
+F 2 "Package_SO:MSOP-8_3x3mm_P0.65mm" H 4200 3000 50  0001 C CNN
 F 3 "" H 4200 3000 50  0001 C CNN
 	1    4200 3000
@@
 F 0 "D1" H 6200 3650 50  0000 C CNN
 F 1 "MAX4477" H 6300 3974 50  0001 C CNN
-F 2 "Package_SO:TSSOP-8_4.4x3mm_P0.65mm" H 6300 3650 50  0001 C CNN
+F 2 "Package_SO:MSOP-8_3x3mm_P0.65mm" H 6300 3650 50  0001 C CNN
 F 3 "" H 6300 3650 50  0001 C CNN
 	2    6300 3650
@@
 	7850 3950 7850 4500
 Wire Wire Line
-	7850 4500 2950 4500
-Wire Wire Line
-	2950 4500 2950 2950
+	7850 4500 3550 4500
 $Comp
 L Device:C C13
@@
 F 3 "" H 3250 3050 50  0001 C CNN
 	1    3250 3050
-	1    0    0    -1
+	-1   0    0    -1
 $EndComp
 Wire Wire Line
@@
 F 3 "http://www.onsemi.com/pub_link/Collateral/NCP1117-D.PDF" H 6300 1500 50  0001 C CNN
 	1    6200 1750
-	1    0    0    -1
+	-1   0    0    -1
 $EndComp
 $Comp
@@
 F 3 "http://www.onsemi.com/pub_link/Collateral/NCP1117-D.PDF" H 3850 1500 50  0001 C CNN
 	1    3750 1750
-	1    0    0    -1
+	-1   0    0    -1
 $EndComp
 Connection ~ 4050 1750
@@
 	2550 4250 3250 4250
 Connection ~ 3250 4250
+Wire Wire Line
+	3550 2950 3550 4500
 $EndSCHEMATC
