File: kicad/Anemometer_200_G473/Anemometer_200_G473.sch (KiCad schematic (older format))
At the start: 86 parts, among them J1 Conn_01x01_Female, J10 Conn_01x01_Female, J11 USB_B_Micro, J12 Conn_01x01_Female, J13 Conn_01x01_Female, J14 Conn_01x01_Female, J15 Conn_01x01_Female, J16 Conn_01x01_Female, J17 Conn_01x01_Female, J18 Conn_01x01_Female, J19 Conn_01x01_Female, J2 Conn_01x01_Female, J20 Conn_01x01_Female, J21 Conn_01x01_Female, J3 Conn_01x08_Shielded, J4 Conn_01x01_Female, J5 Conn_01x01_Female, J6 Conn_01x01_Female, J7 Conn_01x01_Female, J8 Conn_01x04_Shielded, J9 Conn_01x01_Female, U1 W5500, U2 NCP1117-3.3, Y1 16, Y2 Crystal_GND24_Small

Commit message: изменено:      kicad/Amp200_2/Amp200-cache.lib 	изменено:      kicad/Amp200_2/Amp200-rescue.lib 	изменено:      kicad/Amp200_2/Amp200.kicad_pcb 	изменено:      kicad/Amp200_2/Amp200.kicad_pcb-bak 	изменено:      kicad/Amp200_2/Amp200.sch 	изменено:      kicad/Amp200_2/Amp200.sch-bak 	изменено:      kicad/Amp200_2/sym-lib-table 	изменено:      kicad/Anemometer_200_G473/Anemometer_200_G473-cache.lib 	изменено:      kicad/Anemometer_200_G473/Anemometer_200_G473.sch 	изменено:      kicad/Anemometer_200_G473/Anemometer_200_G473.sch-bak 	изменено:      kicad/Anemometer_200_G473/sym-lib-table
Parts:
- removed J10, J12, J14, J9: Conn_01x01_Female, My-library:mini_conn, symbol Connector:Conn_01x01_Female
- added C34, C35: 4.7u, Capacitor_SMD:C_0402_1005Metric, symbol Device:C
- added C36: 6.8n, Capacitor_SMD:C_0402_1005Metric, symbol Device:C
- added C37: CP, symbol Device:CP
- added C? (x10): C, Capacitor_SMD:C_0603_1608Metric, symbol Device:C
- added D10: AD5245, symbol My_Library:AD5245-My_Library
- added D11, D12, D13, D14: D_Zener_Small, symbol Device:D_Zener_Small
- added D9: MAX4477, symbol My_Library:MAX4477
- added J22, J23, J24, J?: Conn_01x01_Female, My-library:mini_conn, symbol Connector:Conn_01x01_Female
- added L3, L?: L, Inductor_SMD:L_0805_2012Metric, symbol Device:L
- added Q1, Q2, Q3, Q4: Q_NMOS_GSD, symbol Device:Q_NMOS_GSD
- added R19, R20, R21, R22, R26, R27, R? (x4): 12.4k, Resistor_SMD:R_0402_1005Metric, symbol Device:R
- added R23, R24, R25, R28, R29: R, Resistor_SMD:R_0603_1608Metric, symbol Device:R
- added U3, U4: TS5A23159DGS, Package_SO:VSSOP-10_3x3mm_P0.5mm, symbol Analog_Switch:TS5A23159DGS
- D2: symbol My_Library:STM32G473CBTx -> Anemometer_200_G473-rescue:STM32G473CBTx-My_Library
- D5: symbol My_Library:CH340N -> Anemometer_200_G473-rescue:CH340N-My_Library
- J3: symbol My_Library:Conn_01x08_Shielded -> Anemometer_200_G473-rescue:Conn_01x08_Shielded-My_Library
- J8: symbol My_Library:Conn_01x04_Shielded -> Anemometer_200_G473-rescue:Conn_01x04_Shielded-My_Library
Connections:
- net labels added: +12v, Analog
- net labels removed: AIn
- wire segments 191 -> 279
- no-connect marks 15 -> 23
Other:
- moved on the sheet: C1, C10, C11, C12, C13, C14, C15, C16, C17, C18, C19, C2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

Commit message: изменено:      kicad/Anemometer_200_G473/Anemometer_200_G473-cache.lib 	изменено:      kicad/Anemometer_200_G473/Anemometer_200_G473.sch 	изменено:      kicad/Anemometer_200_G473/Anemometer_200_G473.sch-bak
Parts:
- added D15, D18, D19, D22: BAT54S, Package_TO_SOT_SMD:SOT-23, symbol Diode:BAT54S
- added D16, D20: BAT54C, Package_TO_SOT_SMD:SOT-23, symbol Diode:BAT54C
- added D17, D21: BAT54A, Package_TO_SOT_SMD:SOT-23, symbol Diode:BAT54A
- added Q5, Q6, Q7, Q8: IRF7343PBF, Package_SO:SOIC-8_3.9x4.9mm_P1.27mm, symbol Transistor_FET:IRF7343PBF
- added R34, R35, R36, R37, R38, R39, R40, R41: 12.4k, Resistor_SMD:R_0402_1005Metric, symbol Device:R
- gave numbers to parts that had none: 16
Connections:
- net at Q1.3 (D), R30.1: no longer J2.1 (Pin_1)
- net at Q2.3 (D), R31.1: no longer J13.1 (Pin_1)
- net at Q3.3 (D), R32.1: no longer J15.1 (Pin_1)
- net at Q4.3 (D), R33.1: no longer J16.1 (Pin_1)
- new net: D17.3, D21.3, Q5.3 (1), Q6.3 (1), Q7.3 (1), Q8.3 (1), R35.1, R37.1, R39.1, R41.1
- new net: D17.1, Q5.4 (G), R35.2
- new net: D15.2, Q5.5 (D), Q5.6 (D)
- new net: D15.1, Q5.1 (S)
- new net: D16.2, Q5.2 (G), R34.1
- new net: D16.3, D20.3, Q5.7 (D), Q5.8 (D), Q6.7 (D), Q6.8 (D), Q7.7 (D), Q7.8 (D), Q8.7 (D), Q8.8 (D), R34.2, R36.2, R38.2, R40.2
- new net: D18.1, Q6.1 (S)
- new net: D16.1, Q6.2 (G), R36.1
- new net: D17.2, Q6.4 (G), R37.2
- new net: D18.2, Q6.5 (D), Q6.6 (D)
- new net: D19.1, Q7.1 (S)
- new net: D20.2, Q7.2 (G), R38.1
- new net: D21.1, Q7.4 (G), R39.2
- new net: D19.2, Q7.5 (D), Q7.6 (D)
- new net: D22.1, Q8.1 (S)
- new net: D20.1, Q8.2 (G), R40.1
- new net: D21.2, Q8.4 (G), R41.2
- new net: D22.2, Q8.5 (D), Q8.6 (D)
- new net: D15.3, J2.1 (Pin_1)
- new net: D18.3, J15.1 (Pin_1)
- new net: D19.3, J13.1 (Pin_1)
- new net: D22.3, J16.1 (Pin_1)
Other:
- moved on the sheet: C38, C39, C40, C41, C42, L4, Q1, Q2, Q3, Q4, R19, R20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
